File: hw/sch_pcb/STEPUPDC02A.kicad_pcb (KiCad board)
At the start: 2 copper layers, 19.8 x 40.1 mm, 18 parts, among them J1 POWER, J2 HEADER_1x02, J4 HEADER_2x04_PARALLEL, M1 HOLE, M2 HOLE, M3 HOLE, M4 HOLE, U1 TPS6104

Commit message: Improve the documentation. a
Other:
- net class Default removed
